File: nixie9v.kicad_pcb (KiCad board)
At the start: 2 copper layers, 86 parts, among them IC1 MC34063AD, IC2 ADUM3221ARZ, IC3 ADUM3221ARZ, IC4 TLP188_TPL,E, IC5 TLP188_TPL,E, IC6 TLP188_TPL,E, IC7 TLP188_TPL,E, J1 Barrel_Jack, J2 USB_B_Micro, J3 UART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

Commit message: upperside
Parts:
- added C19: 0.1u, Capacitor_SMD:C_0603_1608Metric_Pad1.08x0.95mm_HandSolder, F.Cu at (103.9, 73.2)
- added C20: 0.1u, Capacitor_SMD:C_0603_1608Metric_Pad1.08x0.95mm_HandSolder, F.Cu at (95.3, 70.6)
- added C21: 10u, Capacitor_SMD:C_0603_1608Metric_Pad1.08x0.95mm_HandSolder, F.Cu at (89.2, 65.9)
- added C22: 10u, Capacitor_SMD:C_0603_1608Metric_Pad1.08x0.95mm_HandSolder, F.Cu at (91.1, 65.9)
- added C23: 0.1u, Capacitor_SMD:C_0603_1608Metric_Pad1.08x0.95mm_HandSolder, F.Cu at (96.0, 65.9)
- added C24: 0.1u, Capacitor_SMD:C_0603_1608Metric_Pad1.08x0.95mm_HandSolder, F.Cu at (93.1, 65.9)
- D4, D5: footprint Diode_SMD:D_SMF -> Diode_THT:D_DO-41_SOD81_P7.62mm_Horizontal
- moved R23 135.5 mm to (131.8, 36.6), turned to 180 degrees
- moved R24 130.3 mm to (121.7, 36.8), turned to 180 degrees
- moved IC5 125.8 mm to (119.4, 33.0), turned to 180 degrees
- moved R20 124.3 mm to (117.9, 36.8)
- moved IC4 116.2 mm to (129.5, 33.0), turned to 180 degrees
- moved R25 114.2 mm to (111.6, 36.6), turned to 180 degrees
- moved J6 98.9 mm to (128.4, 45.0), turned to -90 degrees
- moved IC6 96.9 mm to (109.2, 33.0), turned to 180 degrees
- moved R21 95.6 mm to (107.8, 36.6)
- moved R26 95.0 mm to (101.5, 36.8), turned to 180 degrees
- moved SW6 91.9 mm to (142.0, 95.5)
- moved U4 91.8 mm to (107.3, 51.6)
- moved R19 89.5 mm to (127.9, 36.6)
- moved R12 88.2 mm to (30.8, 95.5), turned to 180 degrees
- moved IC7 87.5 mm to (99.1, 33.0), turned to 180 degrees
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Connections:
- C6 pad 2: GNDPWR -> GND
- C7 pad 2: GNDPWR -> GND
- R14 pad 1: +5VD -> +3V3
- R16 pad 1: +5VD -> +3V3
- R17 pad 1: +5VD -> +3V3
- R18 pad 1: +5VD -> +3V3
- SW1 pad 1: GND -> GNDPWR
Routing:
- net +3V3: track 0.00 -> 532.0 mm, vias 0 -> 8
- net +5VA: track 0.00 -> 152.2 mm
- net Tube_3: track 0.00 -> 122.1 mm, vias 0 -> 2
- net Tube_2: track 0.00 -> 116.8 mm, vias 0 -> 2
- net NRST: track 0.00 -> 110.7 mm, vias 0 -> 3
- net Tube_1: track 0.00 -> 109.5 mm, vias 0 -> 2
- net USER_SW3: track 0.00 -> 99.6 mm, vias 0 -> 2
- net USER_SW2: track 0.00 -> 93.4 mm, vias 0 -> 2
- net VCC: track 0.00 -> 89.8 mm
- net USER_SW1: track 0.00 -> 83.2 mm, vias 0 -> 2
- net GNDPWR: track 0.00 -> 81.7 mm, vias 0 -> 379
- net GND: track 0.00 -> 81.3 mm, vias 0 -> 311
- net Tube_4: track 0.00 -> 77.2 mm, vias 0 -> 2
- net LED_3: track 0.00 -> 68.5 mm, vias 0 -> 2
- net Net-(D4-Pad2): track 0.00 -> 65.8 mm
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- added copper zone on B.Cu, net GND
- added copper zone on F.Cu, net GND
- added copper zone on B.Cu, net GNDPWR
- added copper zone on F.Cu, net GNDPWR
Other:
- board outline added: 123 x 75 mm

Commit message: accomplished
Changed lines of the file:
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@@
     (pad "4" smd roundrect (at 1.5 1.325 180) (size 0.6 1.55) (layers "F.Cu" "F.Paste" "F.Mask") (roundrect_rratio 0.25)
       (net 6 "+3V3") (pinfunction "Pin_4") (pintype "passive"))
-    (pad "MP" smd roundrect (at -2.8 -1.2 180) (size 1.2 1.8) (layers "F.Cu" "F.Paste" "F.Mask") (roundrect_rratio 0.208333))
-    (pad "MP" smd roundrect (at 2.8 -1.2 180) (size 1.2 1.8) (layers "F.Cu" "F.Paste" "F.Mask") (roundrect_rratio 0.208333))
+    (pad "MP" smd roundrect (at -2.8 -1.2 180) (size 1.2 1.8) (layers "F.Cu" "F.Paste" "F.Mask") (roundrect_rratio 0.2083333333))
+    (pad "MP" smd roundrect (at 2.8 -1.2 180) (size 1.2 1.8) (layers "F.Cu" "F.Paste" "F.Mask") (roundrect_rratio 0.2083333333))
     (model "${KICAD6_3DMODEL_DIR}/Connector_JST.3dshapes/JST_SH_BM04B-SRSS-TB_1x04-1MP_P1.00mm_Vertical.wrl"
       (offset (xyz 0 0 0))
@@
     (pad "4" smd roundrect (at 1.5 1.325 180) (size 0.6 1.55) (layers "F.Cu" "F.Paste" "F.Mask") (roundrect_rratio 0.25)
       (net 11 "NRST") (pinfunction "Pin_4") (pintype "passive"))
-    (pad "MP" smd roundrect (at 2.8 -1.2 180) (size 1.2 1.8) (layers "F.Cu" "F.Paste" "F.Mask") (roundrect_rratio 0.208333))
-    (pad "MP" smd roundrect (at -2.8 -1.2 180) (size 1.2 1.8) (layers "F.Cu" "F.Paste" "F.Mask") (roundrect_rratio 0.208333))
+    (pad "MP" smd roundrect (at 2.8 -1.2 180) (size 1.2 1.8) (layers "F.Cu" "F.Paste" "F.Mask") (roundrect_rratio 0.2083333333))
+    (pad "MP" smd roundrect (at -2.8 -1.2 180) (size 1.2 1.8) (layers "F.Cu" "F.Paste" "F.Mask") (roundrect_rratio 0.2083333333))
     (model "${KICAD6_3DMODEL_DIR}/Connector_JST.3dshapes/JST_SH_BM04B-SRSS-TB_1x04-1MP_P1.00mm_Vertical.wrl"
       (offset (xyz 0 0 0))

Commit message: fix Q3 orietention
Connections:
- Q3 pad 1: GNDPWR -> Net-(D4-Pad1)
- Q3 pad 2: Net-(D4-Pad1) -> GNDPWR
Routing:
- net Net-(D4-Pad1): track 45.8 -> 47.2 mm
Changed lines of the file:
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@@
     (fp_arc (start 1.27 -2.48) (mid 3.561221 -0.949055) (end 3.023625 1.753625) (layer "F.Fab") (width 0.1))
     (pad "1" thru_hole rect (at 0 0) (size 1.3 1.3) (drill 0.75) (layers *.Cu *.Mask)
-      (net 4 "GNDPWR") (pinfunction "E") (pintype "passive"))
+      (net 19 "Net-(D4-Pad1)") (pinfunction "E") (pintype "passive"))
     (pad "2" thru_hole circle (at 1.27 -1.27) (size 1.3 1.3) (drill 0.75) (layers *.Cu *.Mask)
-      (net 19 "Net-(D4-Pad1)") (pinfunction "C") (pintype "passive"))
+      (net 4 "GNDPWR") (pinfunction "C") (pintype "passive"))
     (pad "3" thru_hole circle (at 2.54 0) (size 1.3 1.3) (drill 0.75) (layers *.Cu *.Mask)
       (net 20 "Net-(D4-Pad2)") (pinfunction "B") (pintype "input"))
@@
   (segment (start 113.1805 97.028) (end 115.457 97.028) (width 0.2) (layer "F.Cu") (net 17))
   (segment (start 105.0525 97.028) (end 107.329 97.028) (width 0.2) (layer "F.Cu") (net 18))
+  (segment (start 90.17 53.4162) (end 90.17 47.752) (width 0.762) (layer "B.Cu") (net 19))
+  (segment (start 73.1572 53.4162) (end 90.17 53.4162) (width 0.762) (layer "B.Cu") (net 19))
+  (segment (start 90.17 47.752) (end 90.17 49.6633) (width 0.25) (layer "B.Cu") (net 19))
+  (segment (start 91.874 53.4162) (end 92.89845 52.39175) (width 0.762) (layer "B.Cu") (net 19))
+  (segment (start 90.17 53.4162) (end 91.874 53.4162) (width 0.762) (layer "B.Cu") (net 19))
   (segment (start 59.365 39.624) (end 73.1572 53.4162) (width 0.762) (layer "B.Cu") (net 19))
-  (segment (start 92.52375 50.10575) (end 92.52375 51.12175) (width 0.762) (layer "B.Cu") (net 19))
-  (segment (start 90.17 47.752) (end 92.52375 50.10575) (width 0.762) (layer "B.Cu") (net 19))
-  (segment (start 92.52375 51.12175) (end 94.16845 51.12175) (width 0.762) (layer "B.Cu") (net 19))
-  (segment (start 90.00065 51.12175) (end 92.52375 51.12175) (width 0.762) (layer "B.Cu") (net 19))
-  (segment (start 87.7062 53.4162) (end 90.00065 51.12175) (width 0.762) (layer "B.Cu") (net 19))
-  (segment (start 73.1572 53.4162) (end 87.7062 53.4162) (width 0.762) (layer "B.Cu") (net 19))
   (segment (start 97.536 50.292) (end 97.79 50.038) (width 0.762) (layer "F.Cu") (net 20))
   (segment (start 95.8342 47.752) (end 97.79 47.752) (width 0.762) (layer "F.Cu") (net 20))

Commit message: fix direction tlp188
Parts:
- turned IC4 to 0 degrees
- turned IC5 to 0 degrees
- turned IC6 to 0 degrees
- turned IC7 to 0 degrees
Connections:
- IC4 pad 2: VCC -> Tube_1
- IC4 pad 4: Tube_1 -> VCC
- IC5 pad 2: VCC -> Tube_2
- IC5 pad 4: Tube_2 -> VCC
- IC6 pad 2: VCC -> Tube_3
- IC6 pad 3: Net-(IC6-Pad3) -> Net-(R25-Pad1)
- IC6 pad 4: Tube_3 -> VCC
- IC7 pad 2: VCC -> Tube_4
- IC7 pad 4: Tube_4 -> VCC
- R19 pad 2: Net-(IC4-Pad3) -> Net-(IC4-Pad1)
- R20 pad 2: Net-(IC5-Pad3) -> Net-(IC5-Pad1)
- R21 pad 2: Net-(IC6-Pad3) -> Net-(IC6-Pad1)
- R22 pad 2: Net-(IC7-Pad3) -> Net-(IC7-Pad1)
- R23 pad 1: Net-(IC4-Pad1) -> Net-(IC4-Pad3)
- R24 pad 1: Net-(IC5-Pad1) -> Net-(IC5-Pad3)
- R25 pad 1: Net-(IC6-Pad1) -> Net-(R25-Pad1)
- R26 pad 1: Net-(IC7-Pad1) -> Net-(IC7-Pad3)
Routing:
- net Net-(IC6-Pad3): track 5.97 -> 0.00 mm
- net Net-(IC7-Pad3): track 6.35 -> 2.46 mm
- net Net-(IC7-Pad1): track 2.57 -> 6.35 mm
- net Net-(IC5-Pad3): track 6.17 -> 2.49 mm
- net Net-(IC6-Pad1): track 2.32 -> 5.97 mm
- net Net-(IC4-Pad3): track 5.87 -> 2.23 mm
- net Net-(IC5-Pad1): track 2.56 -> 6.17 mm
- net Net-(IC4-Pad1): track 2.31 -> 5.87 mm
- net Net-(R25-Pad1): track 0.00 -> 2.21 mm
- net Net-(D4-Pad1): track 47.2 -> 45.3 mm
- net Net-(IC1-Pad7): track 27.9 -> 26.8 mm
- net GNDPWR: track 81.7 -> 81.6 mm, vias 379 -> 381
