File: untitled.kicad_sch (KiCad schematic)
At the start: 17 parts, among them IC2 ADUM3221ARZ, IC3 ADUM3221ARZ, IC4 TLP188_TPL,E, IC5 TLP188_TPL,E, IC6 TLP188_TPL,E, IC7 TLP188_TPL,E, J4 Conn_01x10, J5 Conn_01x04, U4 K155NA1

Commit message: add switch and footprint mapping in the middle
Parts:
- J4: footprint (none) -> Connector_PinSocket_2.54mm:PinSocket_1x10_P2.54mm_Vertical
- J5: footprint (none) -> Connector_PinSocket_2.54mm:PinSocket_1x04_P2.54mm_Vertical
- R15, R16, R17, R18, R19, R20, R21, R22: footprint (none) -> Resistor_SMD:R_0603_1608Metric_Pad0.98x0.95mm_HandSolder

Commit message: schema finished
Parts:
- U4: footprint (none) -> SN74141orK155ID1:DIP787W53P279L2176H508Q16N
- renumbered J4 to J5, J5 to J6, R15 to R19, R16 to R20, R17 to R21, R18 to R22, R19 to R23, R20 to R24, R21 to R25, R22 to R26

Commit message: upperside
Parts:
- added C19, C20, C23, C24: 0.1u, Capacitor_SMD:C_0603_1608Metric_Pad1.08x0.95mm_HandSolder, symbol Device:C
- added C21, C22: 10u, Capacitor_SMD:C_0603_1608Metric_Pad1.08x0.95mm_HandSolder, symbol Device:C
Connections:
- net +3V3: now also C19.2, C20.2
- net +5VA: now also C21.2, C22.2, C23.2, C24.2
- net GND: now also C19.1, C20.1
- net GNDPWR: now also C21.1, C22.1, C23.1, C24.1

Commit message: fix direction tlp188
Connections:
- net Tube_1: now also IC4.2 (CATHODE); no longer IC4.4 (COLLECTOR)
- net Tube_2: now also IC5.2 (CATHODE); no longer IC5.4 (COLLECTOR)
- net Tube_3: now also IC6.2 (CATHODE); no longer IC6.4 (COLLECTOR)
- net Tube_4: now also IC7.2 (CATHODE); no longer IC7.4 (COLLECTOR)
- net VCC: now also IC4.4 (COLLECTOR), IC5.4 (COLLECTOR), IC6.4 (COLLECTOR), IC7.4 (COLLECTOR); no longer IC4.2 (CATHODE), IC5.2 (CATHODE), IC6.2 (CATHODE), IC7.2 (CATHODE)
- net at IC7.1 (ANODE): now also R22.2; no longer R26.1
- net at IC7.3 (EMITTER): now also R26.1; no longer R22.2
- net at R24.1: now also IC5.3 (EMITTER); no longer IC5.1 (ANODE)
- net at R23.1: now also IC4.3 (EMITTER); no longer IC4.1 (ANODE)
- net at R20.2: now also IC5.1 (ANODE); no longer IC5.3 (EMITTER)
- net at IC6.1 (ANODE): now also R21.2; no longer R25.1
- net at IC6.3 (EMITTER): now also R25.1; no longer R21.2
- net at R19.2: now also IC4.1 (ANODE); no longer IC4.3 (EMITTER)
Other:
- moved on the sheet: IC4, IC5, IC6, IC7
